File: trunk/Hardware/holter.sch (KiCad schematic (older format))
At the start: 166 parts, among them CN1 2TAP, CN2 2TAP, CN3 3TAP, IC1 256kx8, P1 PROG, P2 EE_PROG, SW1 SW_PUSH, U1 TXB0106, U10 TS5A3159, U11 TS5A3159, U12 ESD_PROTECTOR, U13 ESD_PROTECTOR, U14 ESD_PROTECTOR, U15 ESD_PROTECTOR, U16 ESD_PROTECTOR, U17 ESD_PROTECTOR, U18 ESD_PROTECTOR, U19 ESD_PROTECTOR, U2 TXB0106, U20 ESD_PROTECTOR, U21 ESD_PROTECTOR, U22 ESD_PROTECTOR, U23 ESD_PROTECTOR, U3 TiWi-uB2, U4 STM32F4x1_64, U5 uSD, U6 ADS1298, U7 USBULC6-2M6, U8 USB2641, U9 OPA379, X1 32768, X2 8MHz, X3 24MHz

Commit message: Fix even more typos, arrange parts in the schematic.
---
yaml
---
svn_rev: 4
current_ref: refs/heads/master
current_commit: f7ca86bd98997ffeb8958d9e682c09919540c8bc
head_branch: refs/heads/master
migrated_from: 3
Other:
- note added: "100uA / MHz, USB, SDIO"
- moved on the sheet: ANT1, C1, C10, C11, C12, C13, C132, C133, C134, C135, C136, C137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

Commit message: Accelerometer. Not connected yet.
---
yaml
---
svn_rev: 6
current_ref: refs/heads/master
current_commit: 4e26be5e7ce0dc6a0fababeea61563106a3ee16b
head_branch: refs/heads/master
migrated_from: 3
Parts:
- added C?: 100nF, symbol Csmall
- added C?: 10uF, symbol Csmall
- added U?: LIS2DH12, symbol LIS2DH12
Connections:
- net labels added: ACC_PWR
- wire segments 212 -> 215
Other:
- moved on the sheet: C133, C134, D9, R79, R81, R82
Changed lines of the file:
@@
 LIBS:usbulc6-2m6
 LIBS:rgbled
+LIBS:lis2dh12
 LIBS:holter-cache
 EELAYER 24 0
@@
 L RGBLED D9
 U 1 1 5411FA99
-P 6500 9600
-F 0 "D9" H 6250 9800 39  0000 C CNN
-F 1 "RGBLED" H 6300 9850 39  0000 C CNN
-F 2 "" H 6500 9600 39  0000 C CNN
-F 3 "" H 6500 9600 39  0000 C CNN
-	1    6500 9600
+P 10700 8250
+F 0 "D9" H 10450 8450 39  0000 C CNN
+F 1 "RGBLED" H 10500 8500 39  0000 C CNN
+F 2 "" H 10700 8250 39  0000 C CNN
+F 3 "" H 10700 8250 39  0000 C CNN
+	1    10700 8250
 	1    0    0    -1
 $EndComp
@@
 L +2.8VD #PWR53
 U 1 1 54120635
-P 6500 9200
-F 0 "#PWR53" H 6500 9160 30  0001 C CNN
-F 1 "+2.8VD" H 6500 9310 30  0000 C CNN
-F 2 "" H 6500 9200 60  0000 C CNN
-F 3 "" H 6500 9200 60  0000 C CNN
-	1    6500 9200
+P 10700 7850
+F 0 "#PWR53" H 10700 7810 30  0001 C CNN
+F 1 "+2.8VD" H 10700 7960 30  0000 C CNN
+F 2 "" H 10700 7850 60  0000 C CNN
+F 3 "" H 10700 7850 60  0000 C CNN
+	1    10700 7850
 	1    0    0    -1
 $EndComp
@@
 L R R79
 U 1 1 5412081D
-P 6300 10200
-F 0 "R79" V 6380 10200 40  0000 C CNN
-F 1 "R" V 6307 10201 40  0000 C CNN
-F 2 "" V 6230 10200 30  0000 C CNN
-F 3 "" H 6300 10200 30  0000 C CNN
-	1    6300 10200
+P 10500 8850
+F 0 "R79" V 10580 8850 40  0000 C CNN
+F 1 "R" V 10507 8851 40  0000 C CNN
+F 2 "" V 10430 8850 30  0000 C CNN
+F 3 "" H 10500 8850 30  0000 C CNN
+	1    10500 8850
 	1    0    0    -1
 $EndComp
@@
 L R R81
 U 1 1 54120973
-P 6500 10200
-F 0 "R81" V 6580 10200 40  0000 C CNN
-F 1 "R" V 6507 10201 40  0000 C CNN
-F 2 "" V 6430 10200 30  0000 C CNN
-F 3 "" H 6500 10200 30  0000 C CNN
-	1    6500 10200
+P 10700 8850
+F 0 "R81" V 10780 8850 40  0000 C CNN
+F 1 "R" V 10707 8851 40  0000 C CNN
+F 2 "" V 10630 8850 30  0000 C CNN
+F 3 "" H 10700 8850 30  0000 C CNN
+	1    10700 8850
 	1    0    0    -1
 $EndComp
@@
 L R R82
 U 1 1 54120AC2
-P 6700 10200
-F 0 "R82" V 6780 10200 40  0000 C CNN
-F 1 "R" V 6707 10201 40  0000 C CNN
-F 2 "" V 6630 10200 30  0000 C CNN
-F 3 "" H 6700 10200 30  0000 C CNN
-	1    6700 10200
+P 10900 8850
+F 0 "R82" V 10980 8850 40  0000 C CNN
+F 1 "R" V 10907 8851 40  0000 C CNN
+F 2 "" V 10830 8850 30  0000 C CNN
+F 3 "" H 10900 8850 30  0000 C CNN
+	1    10900 8850
 	1    0    0    -1
 $EndComp
-Text GLabel 6500 10450 3    39   Input ~ 0
+Text GLabel 10700 9100 3    39   Input ~ 0
 R_PWM
-Text GLabel 6300 10450 3    39   Input ~ 0
+Text GLabel 10500 9100 3    39   Input ~ 0
 B_PWM
-Text GLabel 6700 10450 3    39   Input ~ 0
+Text GLabel 10900 9100 3    39   Input ~ 0
 G_PWM
 $Comp
 L C C133
 U 1 1 54125083
-P 7150 9400
-F 0 "C133" H 7150 9500 40  0000 L CNN
-F 1 "10uF" H 7156 9315 40  0000 L CNN
-F 2 "" H 7188 9250 30  0000 C CNN
-F 3 "" H 7150 9400 60  0000 C CNN
-	1    7150 9400
+P 11350 8050
+F 0 "C133" H 11350 8150 40  0000 L CNN
+F 1 "10uF" H 11356 7965 40  0000 L CNN
+F 2 "" H 11388 7900 30  0000 C CNN
+F 3 "" H 11350 8050 60  0000 C CNN
+	1    11350 8050
 	1    0    0    -1
 $EndComp
@@
 L C C134
 U 1 1 5412531B
-P 7400 9400
-F 0 "C134" H 7400 9500 40  0000 L CNN
-F 1 "100nF" H 7406 9315 40  0000 L CNN
-F 2 "" H 7438 9250 30  0000 C CNN
-F 3 "" H 7400 9400 60  0000 C CNN
-	1    7400 9400
+P 11600 8050
+F 0 "C134" H 11600 8150 40  0000 L CNN
+F 1 "100nF" H 11606 7965 40  0000 L CNN
+F 2 "" H 11638 7900 30  0000 C CNN
+F 3 "" H 11600 8050 60  0000 C CNN
+	1    11600 8050
 	1    0    0    -1
 $EndComp
@@
 L GND #PWR57
 U 1 1 541255B5
-P 7150 9600
-F 0 "#PWR57" H 7150 9600 30  0001 C CNN
-F 1 "GND" H 7150 9530 30  0001 C CNN
-F 2 "" H 7150 9600 60  0000 C CNN
-F 3 "" H 7150 9600 60  0000 C CNN
-	1    7150 9600
+P 11350 8250
+F 0 "#PWR57" H 11350 8250 30  0001 C CNN
+F 1 "GND" H 11350 8180 30  0001 C CNN
+F 2 "" H 11350 8250 60  0000 C CNN
+F 3 "" H 11350 8250 60  0000 C CNN
+	1    11350 8250
 	1    0    0    -1
 $EndComp
@@
 L GND #PWR58
 U 1 1 54125705
-P 7400 9600
-F 0 "#PWR58" H 7400 9600 30  0001 C CNN
-F 1 "GND" H 7400 9530 30  0001 C CNN
-F 2 "" H 7400 9600 60  0000 C CNN
-F 3 "" H 7400 9600 60  0000 C CNN
-	1    7400 9600
+P 11600 8250
+F 0 "#PWR58" H 11600 8250 30  0001 C CNN
+F 1 "GND" H 11600 8180 30  0001 C CNN
+F 2 "" H 11600 8250 60  0000 C CNN
+F 3 "" H 11600 8250 60  0000 C CNN
+	1    11600 8250
 	1    0    0    -1
 $EndComp
 Wire Wire Line
-	7400 9200 6500 9200
-Connection ~ 6500 9200
-Connection ~ 7150 9200
+	11600 7850 10700 7850
+Connection ~ 10700 7850
+Connection ~ 11350 7850
 $Comp
 L SW_PUSH SW1
@@
 Text Notes 2900 2850 0    39   ~ 0
 100uA / MHz, USB, SDIO
+$Comp
+L LIS2DH12 U?
+U 1 1 54309490
+P 6550 10000
+F 0 "U?" V 6400 10000 39  0000 C CNN
+F 1 "LIS2DH12" V 6500 10000 39  0000 C CNN
+F 2 "" H 6450 11050 39  0000 C CNN
+F 3 "" H 6450 11050 39  0000 C CNN
+	1    6550 10000
+	1    0    0    -1
+$EndComp
+$Comp
+L GND #PWR?
+U 1 1 54309A80
+P 5750 9850
+F 0 "#PWR?" H 5750 9850 30  0001 C CNN
+F 1 "GND" H 5750 9780 30  0001 C CNN
+F 2 "" H 5750 9850 60  0000 C CNN
+F 3 "" H 5750 9850 60  0000 C CNN
+	1    5750 9850
+	0    1    1    0
+$EndComp
+$Comp
+L GND #PWR?
+U 1 1 54309BDA
+P 5750 9950
+F 0 "#PWR?" H 5750 9950 30  0001 C CNN
+F 1 "GND" H 5750 9880 30  0001 C CNN
+F 2 "" H 5750 9950 60  0000 C CNN
+F 3 "" H 5750 9950 60  0000 C CNN
+	1    5750 9950
+	0    1    1    0
+$EndComp
+$Comp
+L GND #PWR?
+U 1 1 54309DD1
+P 5750 10050
+F 0 "#PWR?" H 5750 10050 30  0001 C CNN
+F 1 "GND" H 5750 9980 30  0001 C CNN
+F 2 "" H 5750 10050 60  0000 C CNN
+F 3 "" H 5750 10050 60  0000 C CNN
+	1    5750 10050
+	0    1    1    0
+$EndComp
+Text GLabel 5450 10250 0    39   Input ~ 0
+ACC_PWR
+$Comp
+L Csmall C?
+U 1 1 5430A2FF
+P 5700 10350
+F 0 "C?" H 5725 10400 30  0000 L CNN
+F 1 "100nF" H 5725 10300 30  0000 L CNN
+F 2 "" H 5700 10350 60  0000 C CNN
+F 3 "" H 5700 10350 60  0000 C CNN
+	1    5700 10350
+	1    0    0    -1
+$EndComp
+$Comp
+L Csmall C?
+U 1 1 5430A472
+P 5500 10350
+F 0 "C?" H 5525 10400 30  0000 L CNN
+F 1 "10uF" H 5525 10300 30  0000 L CNN
+F 2 "" H 5500 10350 60  0000 C CNN
+F 3 "" H 5500 10350 60  0000 C CNN
+	1    5500 10350
+	1    0    0    -1
+$EndComp
+$Comp
+L GND #PWR?
+U 1 1 5430B022
+P 5500 10450
+F 0 "#PWR?" H 5500 10450 30  0001 C CNN
+F 1 "GND" H 5500 10380 30  0001 C CNN
+F 2 "" H 5500 10450 60  0000 C CNN
+F 3 "" H 5500 10450 60  0000 C CNN
+	1    5500 10450
+	1    0    0    -1
+$EndComp
+$Comp
+L GND #PWR?
+U 1 1 5430B180
+P 5700 10450
+F 0 "#PWR?" H 5700 10450 30  0001 C CNN
+F 1 "GND" H 5700 10380 30  0001 C CNN
+F 2 "" H 5700 10450 60  0000 C CNN
+F 3 "" H 5700 10450 60  0000 C CNN
+	1    5700 10450
+	1    0    0    -1
+$EndComp
+Wire Wire Line
+	5750 10250 5450 10250
+Connection ~ 5500 10250
+Connection ~ 5700 10250
+Wire Wire Line
+	5750 10150 5700 10150
+Wire Wire Line
+	5700 10150 5700 10250
+$Comp
+L GND #PWR?
+U 1 1 5430BBCB
+P 5750 9750
+F 0 "#PWR?" H 5750 9750 30  0001 C CNN
+F 1 "GND" H 5750 9680 30  0001 C CNN
+F 2 "" H 5750 9750 60  0000 C CNN
+F 3 "" H 5750 9750 60  0000 C CNN
+	1    5750 9750
+	0    1    1    0
+$EndComp
 $EndSCHEMATC

Commit message: Accelerometer connected.
---
yaml
---
svn_rev: 7
current_ref: refs/heads/master
current_commit: ed49ebf97316f3add3e86dbb4995609e667feb0f
head_branch: refs/heads/master
migrated_from: 3
Parts:
- added R85: 100k, symbol R
- gave numbers to parts that had none: 3
Connections:
- net labels added: ACC_CLK, ACC_CS, ACC_INT, ACC_MISO, ACC_MOSI, EN_2V8
- net labels removed: EN_3V3
- wire segments 215 -> 221
- no-connect marks 33 -> 28
Other:
- note added: "External interrupts:\n C1 - charger\n B9 - button\n A4 - ECG\n C7 - accelerometer"
- moved on the sheet: C132, C133, C134, C138, C139, D9, R10, R79, R80, R81, R82, SW1
